File: PCB/lock-picking.kicad_sch (KiCad schematic)
At the start: 12 parts, among them CN1 B2B-XH-A, CN2 B2B-XH-A, CN3 B2B-XH-A, U1 ESP32-C3-SuperMini, U2 DRV8876PWPR, U3 MLX90393SLW-ABA-011-RE, U4 B4B-XH-A, U5 B4B-XH-A

Commit message: kicad
Parts:
- removed C1, C2: CL10B104KB8NNNC-100nF, EasyEDA:C0603, symbol EasyEDA:CL10B104KB8NNNC
- removed CN2, CN3: B2B-XH-A, EasyEDA:CONN-TH_B2B-XH-A-LF-SN, symbol EasyEDA:B2B-XH-A
- removed R1: ERA2AEB162X, EasyEDA:R0402, symbol EasyEDA:ERA2AEB162X
- removed U4, U5: B4B-XH-A, EasyEDA:CONN-TH_B4B-XH-A-LF-SN, symbol EasyEDA:B4B-XH-A
- added C2, C4: CC0603KRX7R9BB104, EasyEDA:C0603, symbol EasyEDA:CC0603KRX7R9BB104
- added CN4, CN6: XT30APB, EasyEDA:CONN-TH_XT30APB, symbol EasyEDA:XT30APB
- added R2: 0603WAF1501T5E, EasyEDA:R0603, symbol EasyEDA:0603WAF1501T5E
- added U5: AMS1117-5.0, EasyEDA:SOT-223_L6.5-W3.5-P2.30-LS7.0-BR, symbol EasyEDA:AMS1117-5.0
- U1: footprint footprints:ESP32-S3-SuperMini -> ESP32-S3-SuperMini
Connections:
- net 5v: now reaches U1. (3V3), U2.16 (PMODE), U2.3 (nSLEEP), U2.5 (VREF), U3.15 (VDD), U3.2 (SENB/CS), U3.8 (VDD_IO)
- net 5v: now also U5.4 (VOUT)
- net GND: now reaches U1. (3V3), U2.15 (GND), U2.7 (IMODE), U2.9 (PGND), U3.11 (A1), U3.12 (A0), U3.13 (VSS)
- net GND: now also C2.2, CN4.3, CN6.3, R2.1, U5.1 (GND)
- net SCL: now reaches U1.4 (GPIO4)
- net SCL: now also CN4.2, CN6.2
- net SDA: now reaches U1.3 (GPIO3)
- net SDA: now also CN4.1, CN6.1
- net 12v: now reaches U2.11 (VM)
- net 12v: now also C2.1, C4.2, CN4.4, CN6.4, U5.3 (VIN)
- net at U1.5 (GPIO5), U2.6 (IPROPI): now also R2.2
- net at U2.12 (VCP): now also C4.1
- no-connect marks 16 -> 19

Commit message: kicad
Parts:
- added C5, C7: 10uF 25V, Capacitor_SMD:C_0805_2012Metric, symbol Device:C
- added C6: 10uF 16V tant, Capacitor_Tantalum_SMD:CP_EIA-3216-18_Kemet-A, symbol Device:C_Polarized
- added C8, C9: CC0603KRX7R9BB104, EasyEDA:C0603, symbol EasyEDA:CC0603KRX7R9BB104
- added D1: B5819W, Diode_SMD:D_SOD-123, symbol Device:D_Schottky
- added R3, R4: 10k, EasyEDA:R0603, symbol Device:R
- added R5: 10, Resistor_SMD:R_0805_2012Metric, symbol Device:R
- added U4, U6: SMTSOM225BTR, EasyEDA:SMD_BD5.6-D3.6, symbol EasyEDA:SMTSOM225BTR
- U1: value ESP32-C3-SuperMini -> ESP32-S3-SuperMini; footprint ESP32-S3-SuperMini -> footprints:ESP32-S3-SuperMini; symbol ESP32-C3-SuperMini:ESP32-C3-SuperMini -> lock-picking:ESP32-S3-SuperMini
Connections:
- net 12v: now also C7.1, R5.2; no longer U5.3 (VIN)
- net 5v: now also U5.2 (VOUT), C6.1, D1.2 (A); no longer U1. (3V3), U2.16 (PMODE), U2.3 (nSLEEP), U2.5 (VREF), U3.15 (VDD), U3.2 (SENB/CS), U3.8 (VDD_IO)
- net GND: now also U1.GND, U2.17 (EP), C5.2, C6.2, C7.2, C8.1, C9.1; no longer U1. (3V3)
- net SCL: now also U1.3 (GPIO3); no longer U1.4 (GPIO4)
- net SDA: now also U1.4 (GPIO4); no longer U1.3 (GPIO3)
- net IPROPI: now reaches R2.2, U2.6 (IPROPI)
- net IPROPI: now also U1.6 (GPIO6); no longer U1.5 (GPIO5)
- net MAG_SCL: now reaches U1.1 (GPIO1)
- net MAG_SCL: now also U3.3 (SCL/SCLK), R4.2; no longer U3.5 (SDA/MOSI)
- net IN1: now reaches U1.10 (GPIO10)
- net IN1: now also U2.1 (EN/IN1)
- net MAG_SDA: now reaches U1.2 (GPIO2)
- net MAG_SDA: now also U3.5 (SDA/MOSI), R3.2; no longer U3.3 (SCL/SCLK)
- net nFAULT: now reaches U2.4 (nFAULT)
- net nFAULT: now also U1.5 (GPIO5); no longer U1.6 (GPIO6)
- net nSLEEP: now reaches U1.8 (GPIO8)
- net nSLEEP: now also U2.3 (nSLEEP), U2.5 (VREF)
- net IN2: now reaches U1.9 (GPIO9)
- net IN2: now also U2.2 (PH/IN2)
- new net 3v3: C8.2, C9.2, R3.1, R4.1, U1.3V3, U3.15 (VDD), U3.2 (SENB/CS), U3.8 (VDD_IO)
- new net PMODE: U1.12 (GPIO12), U2.16 (PMODE)
- new net VBUS: D1.1 (K), U1.5V
- new net VIN_LDO: C5.1, R5.1, U5.3 (VIN)
- no-connect marks 19 -> 16

Commit message: PCB update (USB C)
Parts:
- removed CN4, CN6: XT30APB, EasyEDA:CONN-TH_XT30APB, symbol EasyEDA:XT30APB
- added U1: HX PZ2.54-1X5P ZZ, EasyEDA:HDR-TH_5P-P2.54-V-M, symbol EasyEDA:HXPZ2.54-1X5PZZ
- added U7: HX TYPE-C 16PIN, EasyEDA:TYPE-C-SMD_HX-TYPE-C-16PIN, symbol EasyEDA:HXTYPE-C16PIN
- renumbered U1 to ESP1
Connections:
- net GND: now also U1.2, U7.A12B1 (GND), U7.B12A1 (GND)
- net IN1: now also ESP1.5 (GPIO5); no longer ESP1.10 (GPIO10)
- net IN2: now also ESP1.4 (GPIO4); no longer ESP1.9 (GPIO9)
- net IPROPI: now also ESP1.2 (GPIO2); no longer ESP1.6 (GPIO6)
- net MAG_SCL: now also ESP1.10 (GPIO10); no longer ESP1.1 (GPIO1)
- net MAG_SDA: now also ESP1.11 (GPIO11); no longer ESP1.2 (GPIO2)
- net PMODE: now also ESP1.6 (GPIO6); no longer ESP1.12 (GPIO12)
- net SCL: now also ESP1.12 (GPIO12), U7.A7 (D-), U7.B7 (D-); no longer ESP1.3 (GPIO3)
- net SDA: now also ESP1.13 (GPIO13), U7.A6 (D+), U7.B6 (D+); no longer ESP1.4 (GPIO4)
- net VBUS: now also U1.1
- net VIN_LDO: now also U7.A9B4 (VBUS), U7.B9A4 (VBUS)
- net nFAULT: now also ESP1.1 (GPIO1); no longer ESP1.5 (GPIO5)
- net nSLEEP: now also ESP1.3 (GPIO3); no longer ESP1.8 (GPIO8)
- net GPIO7: now reaches ESP1.7 (GPIO7)
- net GPIO7: now also U1.5
- new net GPIO8: ESP1.8 (GPIO8), U1.4
- new net GPIO9: ESP1.9 (GPIO9), U1.3
- no-connect marks 16 -> 21
Other:
- note added: "Control Board"
- note added: "Extra Pins"
- note added: "Magnotometer"
- note added: "Motor Driver"
- note added: "USB C"
- note added: "Voltage Regulator"
- moved on the sheet: C2, C3, C4, C5, C6, C7, C8, C9, CN1, D1, R2, R3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
