File: PCB/lock-picking.kicad_pcb (KiCad board)
At the start: 2 copper layers, 34 x 30 mm, 12 parts, among them CN1 B2B-XH-A, CN2 B2B-XH-A, CN3 B2B-XH-A, U1 ESP32-C3-SuperMini, U2 DRV8876PWPR, U3 MLX90393SLW-ABA-011-RE, U4 B4B-XH-A, U5 B4B-XH-A

Commit message: kicad
Parts:
- removed C1: CL10B104KB8NNNC-100nF, EasyEDA:C0603
- removed CN2, CN3: B2B-XH-A, EasyEDA:CONN-TH_B2B-XH-A-LF-SN
- removed R1: ERA2AEB162X, EasyEDA:R0402
- removed U4: B4B-XH-A, EasyEDA:CONN-TH_B4B-XH-A-LF-SN
- added C4: CC0603KRX7R9BB104, EasyEDA:C0603, B.Cu at (35.5, 17.2)
- added CN4: XT30APB, EasyEDA:CONN-TH_XT30APB, F.Cu at (44.0, 30.9)
- added CN6: XT30APB, EasyEDA:CONN-TH_XT30APB, F.Cu at (18.0, 30.9)
- added R2: 0603WAF1501T5E, EasyEDA:R0603, B.Cu at (35.5, 20.8)
- C2: value CL10B104KB8NNNC-100nF -> CC0603KRX7R9BB104
- CN1: moved to B.Cu
- U5: value B4B-XH-A -> AMS1117-5.0; footprint EasyEDA:CONN-TH_B4B-XH-A-LF-SN -> EasyEDA:SOT-223_L6.5-W3.5-P2.30-LS7.0-BR; moved to B.Cu
- moved U5 67.7 mm to (28.1, 28.7), turned to 90 degrees
- moved C2 57.5 mm to (26.0, 20.7), turned to 90 degrees
- moved C3 57.5 mm to (26.0, 17.3)
- moved U1 52.1 mm to (31.0, 27.3)
- moved U3 51.1 mm to (31.0, 37.8)
- moved CN1 49.1 mm to (30.8, 19.0), turned to 180 degrees
- moved U2 48.5 mm to (34.7, 28.0), turned to 0 degrees
Connections:
- C2 pad 1: Net-(U2-VCP) -> 12v
- C2 pad 2: Net-(U2-VM) -> GND
- U1 pad 3: Net-(U1-GPIO3) -> SDA
- U1 pad 4: Net-(U1-GPIO4) -> SCL
- U2 pad 11: Net-(U2-VM) -> 12v
- U2 pad 15: Net-(U1-GND) -> GND
- U2 pad 16: Net-(U1-5V) -> 5v
- U2 pad 3: Net-(U1-5V) -> 5v
- U2 pad 5: Net-(U1-5V) -> 5v
- U2 pad 7: Net-(U1-GND) -> GND
- U2 pad 9: Net-(U1-GND) -> GND
- U3 pad 11: Net-(U1-GND) -> GND
- U3 pad 12: Net-(U1-GND) -> GND
- U3 pad 13: Net-(U1-GND) -> GND
- U3 pad 15: Net-(U1-5V) -> 5v
- U3 pad 2: Net-(U1-5V) -> 5v
- U3 pad 8: Net-(U1-5V) -> 5v
- U5 pad 1: Net-(U1-5V) -> GND
- U5 pad 2: Net-(U1-GND) -> unconnected-(U5-VOUT-Pad2)
- U5 pad 3: Net-(U1-GPIO4) -> 12v
- U5 pad 4: Net-(U1-GPIO3) -> 5v
Routing:
- net Net-(U1-GND): track 88.6 -> 0.00 mm
- net Net-(U1-5V): track 75.3 -> 0.00 mm, vias 4 -> 0
- net GND: track 0.00 -> 70.7 mm, vias 0 -> 1
- net 12v: track 0.00 -> 63.9 mm, vias 0 -> 1
- net SCL: track 0.00 -> 44.7 mm
- net Net-(U2-VM): track 41.3 -> 0.00 mm
- net Net-(U1-GPIO4): track 39.0 -> 0.00 mm
- net Net-(U1-GPIO3): track 38.8 -> 0.00 mm
- net 5v: track 0.00 -> 38.3 mm, vias 0 -> 4
- net SDA: track 0.00 -> 35.0 mm
- net Net-(U2-CPH): track 2.91 -> 21.8 mm
- net Net-(U2-CPL): track 3.22 -> 21.8 mm
- net Net-(U2-OUT1): track 27.9 -> 14.2 mm, vias 0 -> 1
- net Net-(U2-OUT2): track 14.0 -> 19.3 mm, vias 0 -> 1
- net Net-(U2-VCP): track 2.91 -> 0.00 mm
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Other:
- board size 34 x 30 mm -> 34 x 24.7 mm

Commit message: kicad
Parts:
- added C5: 10uF 25V, Capacitor_SMD:C_0805_2012Metric, B.Cu at (36.9, 19.8)
- added C6: 10uF 16V tant, Capacitor_Tantalum_SMD:CP_EIA-3216-18_Kemet-A, B.Cu at (34.8, 30.8)
- added C7: 10uF 25V, Capacitor_SMD:C_0805_2012Metric, B.Cu at (30.0, 34.1)
- added C8: CC0603KRX7R9BB104, EasyEDA:C0603, B.Cu at (28.2, 38.2)
- added C9: CC0603KRX7R9BB104, EasyEDA:C0603, B.Cu at (34.5, 38.6)
- added D1: B5819W, Diode_SMD:D_SOD-123, B.Cu at (25.4, 37.2)
- added R3: 10k, EasyEDA:R0603, B.Cu at (36.0, 35.6)
- added R4: 10k, EasyEDA:R0603, B.Cu at (34.0, 34.9)
- added R5: 10, Resistor_SMD:R_0805_2012Metric, B.Cu at (41.0, 23.7)
- added U4: SMTSOM225BTR, EasyEDA:SMD_BD5.6-D3.6, F.Cu at (18.0, 19.2)
- added U6: SMTSOM225BTR, EasyEDA:SMD_BD5.6-D3.6, F.Cu at (44.0, 19.2)
- U1: value ESP32-C3-SuperMini -> ESP32-S3-SuperMini
- moved C4 16.0 mm to (27.9, 31.3)
- moved C3 13.6 mm to (25.7, 30.9), turned to 0 degrees
- moved C2 12.3 mm to (29.9, 32.4), turned to 0 degrees
- moved U5 7.31 mm to (34.8, 25.6)
- moved U2 7.22 mm to (28.0, 25.4)
- moved R2 2.56 mm to (35.3, 18.2), turned to -90 degrees
Connections:
- R2 pad 2: Net-(U1-GPIO5) -> IPROPI
- U1 pad 1: Net-(U1-GPIO1) -> MAG_SCL
- U1 pad 10: unconnected-(U1-GPIO10-Pad10) -> IN1
- U1 pad 11: (no net) -> unconnected-(U1-GPIO11-Pad11)
- U1 pad 12: (no net) -> PMODE
- U1 pad 13: (no net) -> unconnected-(U1-GPIO13-Pad13)
- U1 pad 2: Net-(U1-GPIO2) -> MAG_SDA
- U1 pad 3: SDA -> SCL
- U1 pad 3V3: (no net) -> 3v3
- U1 pad 4: SCL -> SDA
- U1 pad 5: Net-(U1-GPIO5) -> nFAULT
- U1 pad 5V: (no net) -> VBUS
- U1 pad 6: Net-(U1-GPIO6) -> IPROPI
- U1 pad 8: unconnected-(U1-GPIO8-Pad8) -> nSLEEP
- U1 pad 9: unconnected-(U1-GPIO9-Pad9) -> IN2
- U1 pad GND: (no net) -> GND
- U1 pad RX: (no net) -> unconnected-(U1-GPIO44/RX-PadRX)
- U1 pad TX: (no net) -> unconnected-(U1-GPIO43/TX-PadTX)
- U2 pad 1: unconnected-(U2-EN/IN1-Pad1) -> IN1
- U2 pad 16: 5v -> PMODE
- U2 pad 17: unconnected-(U2-EP-Pad17) -> GND
- U2 pad 2: unconnected-(U2-PH/IN2-Pad2) -> IN2
- U2 pad 3: 5v -> nSLEEP
- U2 pad 4: Net-(U1-GPIO6) -> nFAULT
- U2 pad 5: 5v -> nSLEEP
- U2 pad 6: Net-(U1-GPIO5) -> IPROPI
- U3 pad 15: 5v -> 3v3
- U3 pad 2: 5v -> 3v3
- U3 pad 3: Net-(U1-GPIO2) -> MAG_SCL
- U3 pad 5: Net-(U1-GPIO1) -> MAG_SDA
- U3 pad 8: 5v -> 3v3
- U5 pad 2: unconnected-(U5-VOUT-Pad2) -> 5v
- U5 pad 3: 12v -> VIN_LDO
Routing:
- net GND: track 70.7 -> 32.7 mm, vias 1 -> 10
- net 12v: track 63.9 -> 37.1 mm
- net 3v3: track 0.00 -> 23.7 mm, vias 0 -> 3
- net 5v: track 38.3 -> 16.4 mm, vias 4 -> 2
- net Net-(U2-CPH): track 21.8 -> 2.09 mm
- net Net-(U2-CPL): track 21.8 -> 3.10 mm
- net IPROPI: track 0.00 -> 16.7 mm, vias 0 -> 2
- net nFAULT: track 0.00 -> 14.3 mm, vias 0 -> 1
- net MAG_SDA: track 0.00 -> 14.0 mm
- net nSLEEP: track 0.00 -> 11.2 mm
- net Net-(U1-GPIO2): track 11.2 -> 0.00 mm
- net SDA: track 35.0 -> 45.7 mm, vias 0 -> 1
- net Net-(U2-OUT1): track 14.2 -> 3.67 mm, vias 1 -> 0
- net Net-(U1-GPIO6): track 9.98 -> 0.00 mm
- net Net-(U1-GPIO5): track 9.26 -> 0.00 mm, vias 1 -> 0
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- added copper zone on B.Cu, net 5v
- added copper zone on B.Cu, net GND
- added copper zone on F.Cu, net GND
Other:
- outline, holes or cut-outs redrawn

Commit message: PCB update (USB C)
Parts:
- removed CN4, CN6: XT30APB, EasyEDA:CONN-TH_XT30APB
- added ESP1: ESP32-S3-SuperMini, footprints:ESP32-S3-SuperMini, F.Cu at (31.0, 31.5)
- added U7: HX TYPE-C 16PIN, EasyEDA:TYPE-C-SMD_HX-TYPE-C-16PIN, F.Cu at (30.5, 19.2)
- U1: value ESP32-S3-SuperMini -> HX PZ2.54-1X5P ZZ; footprint footprints:ESP32-S3-SuperMini -> EasyEDA:HDR-TH_5P-P2.54-V-M
- moved C2 54.3 mm to (80.4, 52.3)
- moved C4 54.3 mm to (78.4, 51.2)
- moved D1 54.3 mm to (75.9, 57.1)
- moved C3 54.3 mm to (76.2, 50.8)
- moved C6 54.3 mm to (85.2, 50.7)
- moved C7 54.3 mm to (80.5, 54.0)
- moved C8 54.3 mm to (78.7, 58.1)
- moved C9 54.3 mm to (85.0, 58.5)
- moved R3 54.3 mm to (86.5, 55.5)
- moved R4 54.3 mm to (84.5, 54.8)
- moved R5 54.3 mm to (91.5, 43.6)
- moved U1 54.3 mm to (81.5, 47.2)
- moved U2 54.3 mm to (78.5, 45.2)
- moved U3 54.3 mm to (81.5, 57.6)
- moved U5 54.3 mm to (85.2, 45.5)
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Connections:
- U1 pad 1: MAG_SCL -> VBUS
- U1 pad 2: MAG_SDA -> GND
- U1 pad 3: SCL -> GPIO9
- U1 pad 4: SDA -> GPIO8
- U1 pad 5: nFAULT -> GPIO7
Routing:
- net Net-(U2-OUT1): track 3.67 -> 29.7 mm, vias 0 -> 2
- net GND: track 32.7 -> 6.61 mm, vias 10 -> 5
- net 3v3: track 23.7 -> 0.00 mm, vias 3 -> 0
- net IN2: track 4.57 -> 23.7 mm, vias 0 -> 3
- net unconnected-(U7-EH-Pad20): track 0.00 -> 6.91 mm
- net 12v: track 37.1 -> 33.5 mm
- net GPIO8: track 0.00 -> 3.54 mm
- net VBUS: track 2.49 -> 0.00 mm
- net nFAULT: track 14.3 -> 16.8 mm, vias 1 -> 2
- net IN1: track 2.34 -> 0.00 mm, vias 0 -> 1
- net unconnected-(U7-EH-Pad19): vias 0 -> 1
Other:
- board size 34 x 24.7 mm -> 34 x 25.4 mm

Commit message: PCB updates
Parts:
- removed CN1: B2B-XH-A, EasyEDA:CONN-TH_B2B-XH-A-LF-SN
- added U8: AMS1117-5.0_C347223, EasyEDA:SOT-223_L6.7-W3.5-P2.30-BR, F.Cu at (23.8, 28.4)
- U5: value AMS1117-5.0 -> S2B-PH-K-S; footprint EasyEDA:SOT-223_L6.5-W3.5-P2.30-LS7.0-BR -> EasyEDA:CONN-TH_S2B-PH-K-S-LF-SN; moved to F.Cu
- U7: moved to B.Cu
- moved C9 74.5 mm to (16.4, 29.2)
- moved U5 73.8 mm to (17.5, 16.4), turned to 0 degrees
- moved R3 72.5 mm to (21.0, 24.5), turned to 180 degrees
- moved U3 72.0 mm to (17.1, 25.4)
- moved R5 71.2 mm to (24.5, 19.5), turned to 90 degrees
- moved R4 69.6 mm to (21.0, 26.2), turned to 180 degrees
- moved C4 68.0 mm to (18.2, 19.5)
- moved C8 67.9 mm to (16.3, 31.2), turned to 180 degrees
- moved C6 64.2 mm to (24.9, 29.0)
- moved C2 64.1 mm to (19.8, 31.5)
- moved U2 62.8 mm to (23.5, 15.0), turned to 90 degrees
- moved U1 62.0 mm to (20.8, 34.5), turned to 0 degrees
- moved C7 61.9 mm to (24.9, 26.8), turned to 180 degrees
- moved C3 59.0 mm to (26.2, 19.4), turned to 90 degrees
- moved D1 57.2 mm to (24.5, 32.0), turned to 180 degrees
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Connections:
- U5 pad 1: GND -> Net-(U2-OUT2)
- U5 pad 2: 5v -> Net-(U2-OUT1)
Routing:
- net SDA: track 45.7 -> 0.00 mm, vias 1 -> 0
- net SCL: track 43.0 -> 0.00 mm, vias 1 -> 0
- net 12v: track 33.5 -> 0.00 mm, vias 1 -> 0
- net Net-(U2-OUT1): track 29.7 -> 0.00 mm, vias 2 -> 0
- net IN2: track 23.7 -> 0.00 mm, vias 3 -> 0
- net nFAULT: track 16.8 -> 0.00 mm, vias 2 -> 0
- net IPROPI: track 16.7 -> 0.00 mm, vias 2 -> 0
- net 5v: track 16.4 -> 0.00 mm, vias 2 -> 0
- net Net-(U2-OUT2): track 14.2 -> 0.00 mm, vias 1 -> 0
- net MAG_SDA: track 14.0 -> 0.00 mm
- net nSLEEP: track 11.2 -> 0.00 mm
- net MAG_SCL: track 8.73 -> 0.00 mm
- net unconnected-(U7-EH-Pad20): track 6.91 -> 0.00 mm
- net GND: track 6.61 -> 0.00 mm, vias 5 -> 0
- net VIN_LDO: track 3.61 -> 0.00 mm
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- removed copper zone on B.Cu, net 5v
- removed copper zone on B.Cu, net GND
- removed copper zone on F.Cu, net GND
Other:
- board size 34 x 25.4 mm -> 25 x 24 mm

Commit message: PCB routing
Parts:
- removed ESP1: ESP32-S3-SuperMini, footprints:ESP32-S3-SuperMini
- removed R5: 10, Resistor_SMD:R_0805_2012Metric
- removed U5: S2B-PH-K-S, EasyEDA:CONN-TH_S2B-PH-K-S-LF-SN
- removed U6: SMTSOM225BTR, EasyEDA:SMD_BD5.6-D3.6
- removed U7: HX TYPE-C 16PIN, EasyEDA:TYPE-C-SMD_HX-TYPE-C-16PIN
- removed U8: AMS1117-5.0_C347223, EasyEDA:SOT-223_L6.7-W3.5-P2.30-BR
- added C1: 10uF 25V, Capacitor_SMD:C_0805_2012Metric, B.Cu at (25.1, 34.4)
- added C10: 100nF 16V, Capacitor_SMD:C_0402_1005Metric, B.Cu at (19.8, 26.4)
- added C11: 10uF 6.3V, Capacitor_SMD:C_0402_1005Metric, B.Cu at (15.7, 28.9)
- added C12: 10nF 50V, Capacitor_SMD:C_0402_1005Metric, B.Cu at (22.0, 22.1)
- added H1: M2 SMD nut, Library:M2_SMD_nut_SMTSOM225_ring4.2, F.Cu at (33.3, 15.3)
- added H2: M2 SMD nut, Library:M2_SMD_nut_SMTSOM225_ring4.2, F.Cu at (33.3, 32.4)
- added J1: USB-C 16P (12V + I2C), Library:USB-C_HX-TYPE-C-16PIN_NPTH-pegs, B.Cu at (33.4, 23.9)
- added J2: Motor (JST-PH 2P), EasyEDA:CONN-TH_S2B-PH-K-S-LF-SN, F.Cu at (19.2, 17.3)
- added L1: 4.7uH, Inductor_SMD:L_Changjiang_FTC252012S, B.Cu at (20.1, 31.5)
- added R1: 1.5k 1%, Resistor_SMD:R_0402_1005Metric, B.Cu at (22.0, 21.0)
- added TP1: Pad, TestPoint:TestPoint_Pad_D1.5mm, F.Cu at (21.1, 30.8)
- added TP2: Pad, TestPoint:TestPoint_Pad_D1.5mm, F.Cu at (18.6, 30.8)
- added TP3: Pad, TestPoint:TestPoint_Pad_D1.5mm, F.Cu at (24.9, 34.0)
- added TP4: Pad, TestPoint:TestPoint_Pad_D1.5mm, F.Cu at (22.4, 34.0)
- added TP5: Pad, TestPoint:TestPoint_Pad_D1.5mm, F.Cu at (23.6, 30.8)
- added TP6: Pad, TestPoint:TestPoint_Pad_D1.5mm, F.Cu at (17.3, 34.0)
- added TP7: Pad, TestPoint:TestPoint_Pad_D1.5mm, F.Cu at (19.8, 34.0)
- C2, C9: value CC0603KRX7R9BB104 -> 100nF 16V; footprint EasyEDA:C0603 -> Capacitor_SMD:C_0402_1005Metric
- C3: value CL10B223KB8NNNC-22nF -> 47uF 6.3V; footprint EasyEDA:C0603 -> Capacitor_SMD:C_0805_2012Metric
- C4: value CC0603KRX7R9BB104 -> 47uF 6.3V; footprint EasyEDA:C0603 -> Capacitor_SMD:C_0805_2012Metric
- C5: value 10uF 25V -> 100nF 50V; footprint Capacitor_SMD:C_0805_2012Metric -> Capacitor_SMD:C_0402_1005Metric
- C6: value 10uF 16V tant -> 22uF 25V; footprint Capacitor_Tantalum_SMD:CP_EIA-3216-18_Kemet-A -> Capacitor_SMD:C_1206_3216Metric
- C7: value 10uF 25V -> 100nF 16V; footprint Capacitor_SMD:C_0805_2012Metric -> Capacitor_SMD:C_0402_1005Metric
- C8: value CC0603KRX7R9BB104 -> 22nF 50V; footprint EasyEDA:C0603 -> Capacitor_SMD:C_0402_1005Metric
- D1: value B5819W -> 1N5819WS; footprint Diode_SMD:D_SOD-123 -> Diode_SMD:D_SOD-323
- R2: value 0603WAF1501T5E -> 10k; footprint EasyEDA:R0603 -> Resistor_SMD:R_0402_1005Metric
- R3, R4: value 10k -> 2.2k; footprint EasyEDA:R0603 -> Resistor_SMD:R_0402_1005Metric
- U1: value HX PZ2.54-1X5P ZZ -> ESP32-S3-SuperMini; footprint EasyEDA:HDR-TH_5P-P2.54-V-M -> footprints:ESP32-S3-SuperMini
- U2: value DRV8876PWPR -> DRV8876RGTR; footprint EasyEDA:HTSSOP-16_L5.0-W4.4-P0.65-LS6.4-BL-EP -> Library:QFN-16-1EP_3x3mm_P0.5mm_EP1.68x1.68mm_ThermalVias0.3
- U4: value SMTSOM225BTR -> AP63205WU-7; footprint EasyEDA:SMD_BD5.6-D3.6 -> Package_TO_SOT_SMD:TSOT-23-6; moved to B.Cu
- moved C8 19.9 mm to (25.2, 13.4), turned to 0 degrees
- moved U4 18.2 mm to (25.1, 31.5), turned to 180 degrees
- moved C6 17.0 mm to (17.9, 13.5), turned to 180 degrees
- moved C3 16.1 mm to (20.8, 34.5), turned to 0 degrees
- moved C4 15.0 mm to (17.1, 34.5), turned to 180 degrees
- moved C7 13.4 mm to (23.2, 13.4)
- moved U1 10.7 mm to (21.1, 23.9), turned to 180 degrees
- moved D1 8.21 mm to (16.3, 32.4), turned to 0 degrees
- moved C9 7.67 mm to (15.4, 21.6), turned to -90 degrees
- moved R4 6.09 mm to (17.6, 21.2)
- moved C5 6.07 mm to (21.3, 13.4), turned to 180 degrees
- moved R2 3.72 mm to (23.9, 19.1), turned to 180 degrees
- moved C2 2.74 mm to (22.5, 31.0), turned to 90 degrees
- moved U2 1.40 mm to (23.9, 16.3)
- moved R3 1.25 mm to (19.8, 24.4), turned to -90 degrees
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Connections:
- C2 pad 1: 12v -> Net-(U4-SW)
- C2 pad 2: GND -> Net-(U4-BST)
- C3 pad 1: Net-(U2-CPL) -> +5V
- C3 pad 2: Net-(U2-CPH) -> GND
- C4 pad 1: Net-(U2-VCP) -> +5V
- C4 pad 2: 12v -> GND
- C5 pad 1: VIN_LDO -> +12V
- C6 pad 1: 5v -> +12V
- C7 pad 1: 12v -> /DRV_VCP
- C7 pad 2: GND -> +12V
- C8 pad 1: GND -> /DRV_CPH
- C8 pad 2: 3v3 -> /DRV_CPL
- C9 pad 1: GND -> +3V3
- C9 pad 2: 3v3 -> GND
- D1 pad 2: 5v -> +5V
- R2 pad 1: GND -> /DRV_nFAULT
- R2 pad 2: IPROPI -> +3V3
- R3 pad 1: 3v3 -> /MAG_SDA
- R3 pad 2: MAG_SDA -> +3V3
- R4 pad 1: 3v3 -> /MAG_SCL
- R4 pad 2: MAG_SCL -> +3V3
- U1 pad 1: VBUS -> /DRV_IPROPI
- U1 pad 2: GND -> /DRV_nFAULT
- U1 pad 3: GPIO9 -> /I2C_SDA
- U1 pad 4: GPIO8 -> /I2C_SCL
- U1 pad 5: GPIO7 -> /DRV_nSLEEP
- U2 pad 1: IN1 -> /DRV_nSLEEP
- U2 pad 10: Net-(U2-OUT2) -> /DRV_VCP
- U2 pad 11: 12v -> /DRV_CPH
- U2 pad 12: Net-(U2-VCP) -> /DRV_CPL
- U2 pad 13: Net-(U2-CPH) -> GND
- U2 pad 14: Net-(U2-CPL) -> GND
- U2 pad 15: GND -> /DRV_IN1_EN
- U2 pad 16: PMODE -> /DRV_IN2_PH
- U2 pad 2: IN2 -> /DRV_nFAULT
- U2 pad 3: nSLEEP -> +3V3
- U2 pad 4: nFAULT -> /DRV_IPROPI
- U2 pad 5: nSLEEP -> GND
- U2 pad 6: IPROPI -> /MOT_OUT1
- U2 pad 8: Net-(U2-OUT1) -> /MOT_OUT2
- U2 pad 9: GND -> +12V
- U3 pad 1: unconnected-(U3-INT-Pad1) -> /MAG_INT
- U3 pad 10: unconnected-(U3-N/C-Pad10) -> GND
- U3 pad 14: unconnected-(U3-N/C-Pad14) -> GND
- U3 pad 15: 3v3 -> +3V3
- U3 pad 16: unconnected-(U3-N/C-Pad16) -> GND
- U3 pad 17: unconnected-(U3-EP-Pad17) -> GND
- U3 pad 2: 3v3 -> +3V3
- U3 pad 3: MAG_SCL -> /MAG_SCL
- U3 pad 4: unconnected-(U3-N/C-Pad4) -> GND
- U3 pad 5: MAG_SDA -> /MAG_SDA
- U3 pad 8: 3v3 -> +3V3
- U3 pad 9: unconnected-(U3-N/C-Pad9) -> GND
- U4 pad 1: unconnected-(U4-Pad1)_1 -> +5V
Routing:
- net +3V3: track 0.00 -> 40.8 mm, vias 0 -> 3
- net GND: track 0.00 -> 26.1 mm, vias 0 -> 25
- net +12V: track 0.00 -> 22.9 mm, vias 0 -> 7
- net /DRV_IPROPI: track 0.00 -> 16.8 mm
- net /MAG_SDA: track 0.00 -> 14.1 mm
- net /EXP_IO12: track 0.00 -> 13.4 mm
- net +5V: track 0.00 -> 13.2 mm
- net /DRV_nFAULT: track 0.00 -> 11.7 mm
- net /MAG_SCL: track 0.00 -> 8.57 mm
- net /EXP_IO13: track 0.00 -> 8.53 mm
- net /EXP_RX: track 0.00 -> 7.91 mm
- net VBUS: track 0.00 -> 6.21 mm
- net /MOT_OUT2: track 0.00 -> 5.63 mm
- net /DRV_IN1_EN: track 0.00 -> 5.45 mm
- net /I2C_SCL: track 0.00 -> 4.78 mm
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- added copper zone on F.Cu, net +12V
- added copper zone on B.Cu, net GND
- added copper zone on F.Cu, net GND
Other:
- board size 25 x 24 mm -> 25 x 23.7 mm
- board text added: "3V3"
- board text added: "5V"
- board text added: "ESP socket keep out"
- board text added: "GND"
- board text added: "IO12"
- board text added: "IO13"
- board text added: "ROUTING NOTES rev 3b (2 layers, routed + poured, reviewed) Frame origin = board top-left (abs 12,12). Board 25.0 x 23.7, 1 mm corner radius. 1 BACK = every PCBA part + most signals. FRONT = GND pour, a 12 V copper area, short hops. 2 12 V: J1 top VBUS pad -> 3 vias -> front 12 V copper (gaps between ESP pins 6/5 and 5/4) -> inside the right header -> along the top edge -> 3 vias -> C5/C7/U2 VM. N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"
- board text added: "RX"
- board text added: "TX"
