File: PCB/main board/lock-picking.kicad_sch (KiCad schematic)
At the start: 33 parts, among them J1 USB-C 16P (12V + I2C), J2 Motor (JST-PH 2P), U1 ESP32-S3-SuperMini, U2 DRV8876RGTR, U3 MLX90393SLW-ABA-011-RE, U4 AP63205WU-7

Commit message: re-organised
Parts:
- added TP10, TP11: Pad, TestPoint:TestPoint_Pad_D1.0mm, symbol Connector:TestPoint
- added TP8, TP9: Pad, TestPoint:TestPoint_Pad_D1.5mm, symbol Connector:TestPoint
Connections:
- net +12V: now also TP8.1
- net +5V: now also TP10.1
- net GND: now also TP11.1, TP9.1
Other:
- note added: "PROBE PADS"
