File: PCB/main board/lock-picking.kicad_pcb (KiCad board)
At the start: 2 copper layers, 25 x 23.7 mm, 33 parts, among them J1 USB-C 16P (12V + I2C), J2 Motor (JST-PH 2P), U1 ESP32-S3-SuperMini, U2 DRV8876RGTR, U3 MLX90393SLW-ABA-011-RE, U4 AP63205WU-7

Commit message: re-organised
Parts:
- added TP10: Pad, TestPoint:TestPoint_Pad_D1.0mm, B.Cu at (20.2, 28.9)
- added TP11: Pad, TestPoint:TestPoint_Pad_D1.0mm, B.Cu at (17.7, 28.9)
- added TP8: Pad, TestPoint:TestPoint_Pad_D1.5mm, F.Cu at (35.2, 22.6)
- added TP9: Pad, TestPoint:TestPoint_Pad_D1.5mm, F.Cu at (35.2, 25.1)
Routing:
- net GND: track 26.1 -> 29.2 mm
- net +5V: track 13.2 -> 14.3 mm
Other:
- board text added: "12V"

Commit message: PCB
Parts:
- moved C11 7.28 mm to (15.4, 21.6), turned to -90 degrees
- moved TP10 4.74 mm to (24.9, 28.8)
- moved TP11 4.74 mm to (22.4, 28.8)
- moved C9 3.50 mm to (15.4, 25.1)
- moved U3 3.50 mm to (17.1, 28.1)
- moved C10 2.25 mm to (19.6, 28.6), turned to 90 degrees
- moved R3 1.50 mm to (19.8, 25.9), turned to 0 degrees
Routing:
- net +3V3: track 40.8 -> 46.6 mm
- net /MAG_SCL: track 8.57 -> 12.1 mm
- net /MAG_INT: track 4.14 -> 7.64 mm
- net /MAG_SDA: track 14.1 -> 16.9 mm
- net GND: track 29.2 -> 30.0 mm
Other:
- outline, holes or cut-outs redrawn
- board text added: "ROUTING NOTES rev 3c (2 layers, routed + poured, reviewed) Frame origin = board top-left (abs 12,12). Board 25.0 x 23.7, 1 mm corner radius. 1 BACK = every PCBA part + most signals. FRONT = GND pour, a 12 V copper area, short hops. 2 12 V: J1 top VBUS pad -> 3 vias -> front 12 V copper (gaps between ESP pins 6/5 and 5/4) -> inside the right header -> along the top edge -> 3 vias -> C5/C7/U2 VM. N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"
- board text removed: "ROUTING NOTES rev 3b (2 layers, routed + poured, reviewed) Frame origin = board top-left (abs 12,12). Board 25.0 x 23.7, 1 mm corner radius. 1 BACK = every PCBA part + most signals. FRONT = GND pour, a 12 V copper area, short hops. 2 12 V: J1 top VBUS pad -> 3 vias -> front 12 V copper (gaps between ESP pins 6/5 and 5/4) -> inside the right header -> along the top edge -> 3 vias -> C5/C7/U2 VM. N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"
