File: PCB/main-board/main-board.kicad_pcb (KiCad board)
At the start: 2 copper layers, 25 x 23.7 mm, 37 parts, among them J1 USB-C 16P (12V + I2C), J2 Motor (JST-PH 2P), U1 ESP32-S3-SuperMini, U2 DRV8876RGTR, U3 MLX90393SLW-ABA-011-RE, U4 AP63205WU-7

Commit message: PCB stuff
Parts:
- removed TP10, TP11: Pad, TestPoint:TestPoint_Pad_D1.0mm
- added C13: 100nF 16V, Capacitor_SMD:C_0402_1005Metric, B.Cu at (21.8, 25.3)
- added JP1: D+ select, Jumper:SolderJumper-3_P1.3mm_Bridged12_RoundedPad1.0x1.5mm, F.Cu at (25.9, 24.7)
- added JP2: D- select, Jumper:SolderJumper-3_P1.3mm_Bridged12_RoundedPad1.0x1.5mm, F.Cu at (25.9, 22.0)
- added JP3: RX link, Jumper:SolderJumper-2_P1.3mm_Bridged_RoundedPad1.0x1.5mm, F.Cu at (20.6, 19.5)
- added JP4: 120R term, Jumper:SolderJumper-2_P1.3mm_Open_RoundedPad1.0x1.5mm, F.Cu at (17.1, 19.5)
- added R5: 120R, Resistor_SMD:R_0402_1005Metric, B.Cu at (16.1, 16.9)
- added R6: 10k, Resistor_SMD:R_0402_1005Metric, B.Cu at (18.0, 24.4)
- added U5: SN65HVD230, Package_SO:SOIC-8_3.9x4.9mm_P1.27mm, F.Cu at (19.7, 25.9)
- J1: value USB-C 16P (12V + I2C) -> USB-C 16P (12V + CAN/I2C)
- moved TP9 1.11 mm to (35.2, 26.2)
- moved TP8 1.10 mm to (35.2, 21.5)
- moved J2 1.04 mm to (19.2, 16.2)
- moved C12 0.15 mm to (22.0, 22.2)
Connections:
- J1 pad A6: /I2C_SDA -> /BUS_P
- J1 pad A7: /I2C_SCL -> /BUS_N
- J1 pad B6: /I2C_SDA -> /BUS_P
- J1 pad B7: /I2C_SCL -> /BUS_N
- U1 pad 3: /I2C_SDA -> /SDA_CANTX
- U1 pad 4: /I2C_SCL -> /SCL_CANRX
Routing:
- net +12V: track 22.9 -> 53.5 mm
- net /CANH: track 0.00 -> 21.8 mm, vias 0 -> 2
- net /CANL: track 0.00 -> 17.3 mm, vias 0 -> 1
- net GND: track 30.0 -> 44.0 mm, vias 25 -> 20
- net /SDA_CANTX: track 0.00 -> 9.74 mm
- net /BUS_N: track 0.00 -> 9.67 mm, vias 0 -> 1
- net /SCL_CANRX: track 0.00 -> 9.05 mm
- net /CAN_RS: track 0.00 -> 8.92 mm, vias 0 -> 1
- net /BUS_P: track 0.00 -> 8.90 mm, vias 0 -> 1
- net /CAN_RXD: track 0.00 -> 7.48 mm, vias 0 -> 2
- net /I2C_SCL: track 4.78 -> 0.00 mm
- net Net-(JP4-B): track 0.00 -> 3.86 mm, vias 0 -> 1
- net /I2C_SDA: track 2.72 -> 0.00 mm
- net +3V3: track 46.6 -> 48.5 mm
- net /DRV_nFAULT: track 12.1 -> 13.4 mm
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- removed copper zone on F.Cu, net +12V
Other:
- outline, holes or cut-outs redrawn
- board text added: "CAN"
- board text added: "I2C"
- board text added: "RX CAN"
- board text added: "TERM"

Commit message: PCB dev
Parts:
- removed J1: USB-C 16P (12V + CAN/I2C), main-board:USB-C_HX-TYPE-C-16PIN_NPTH-pegs
- removed TP8, TP9: Pad, TestPoint:TestPoint_Pad_D1.5mm
- added CN2: XT30APB, main-board:CONN-TH_XT30APB, F.Cu at (39.6, 33.7)
- added R7: 10k, Resistor_SMD:R_0402_1005Metric, B.Cu at (27.9, 38.0)
- moved H2 13.8 mm to (39.6, 44.6)
- moved TP5 12.1 mm to (30.0, 41.0)
- moved TP1 12.0 mm to (27.2, 41.0)
- moved TP2 11.9 mm to (24.7, 41.0)
- moved C11 11.4 mm to (21.6, 31.3)
- moved C12 11.4 mm to (28.1, 31.9)
- moved C13 11.4 mm to (27.9, 34.9)
- moved C7 11.4 mm to (29.4, 23.1)
- moved C8 11.4 mm to (31.3, 23.1)
- moved R2 11.4 mm to (30.1, 28.8)
- moved C1 11.4 mm to (31.2, 44.0)
- moved C2 11.4 mm to (28.6, 40.7)
- moved C3 11.4 mm to (26.9, 44.1)
- moved C4 11.4 mm to (23.2, 44.1)
- moved C5 11.4 mm to (27.4, 23.1)
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Routing:
- net /BUS_N: track 9.67 -> 17.8 mm, vias 1 -> 2
- net GND: track 44.0 -> 38.9 mm, vias 20 -> 18
- net /SDA_CANTX: track 9.74 -> 11.7 mm, vias 0 -> 1
- net /BUS_P: track 8.90 -> 10.7 mm, vias 1 -> 2
- net +12V: track 53.5 -> 52.5 mm, vias 7 -> 3
- net /MAG_SDA: track 16.9 -> 16.2 mm
Other:
- board size 25 x 23.7 mm -> 24.7 x 28.4 mm

Commit message: new schematic
Parts:
- removed TP3, TP4: Pad, TestPoint:TestPoint_Pad_D1.5mm
- added C14: 47pF 50V, Capacitor_SMD:C_0402_1005Metric, F.Cu at (81.1, 68.2)
- added IO7: Pad, TestPoint:TestPoint_Pad_D1.5mm, F.Cu at (22.0, 43.8)
- added R8: 75k, Resistor_SMD:R_0402_1005Metric, F.Cu at (78.2, 68.2)
- added R9: 10k, Resistor_SMD:R_0402_1005Metric, F.Cu at (78.2, 70.2)
- L1: value 4.7uH -> 10uH
- R1: value 1.5k 1% -> 3.3k; footprint Resistor_SMD:R_0402_1005Metric -> Resistor_SMD:R_0805_2012Metric_Pad1.20x1.40mm_HandSolder
- U4: value AP63205WU-7 -> TPS54202DDCR
- moved C5 95.4 mm to (121.5, 39.0)
- moved C6 92.1 mm to (115.5, 34.2)
- moved R2 90.2 mm to (120.0, 35.0)
- moved C7 90.1 mm to (118.3, 37.2)
- moved C8 90.1 mm to (120.3, 37.2)
- moved D1 89.5 mm to (106.0, 74.0)
- moved L1 82.6 mm to (102.0, 74.0)
- moved C11 81.5 mm to (96.1, 64.2)
- moved C9 81.5 mm to (96.1, 67.7)
- moved R4 81.5 mm to (98.2, 63.7)
- moved R6 81.5 mm to (98.6, 66.9)
- moved R1 79.3 mm to (102.0, 59.5)
- moved U5 78.8 mm to (104.3, 43.1)
- moved C10 73.4 mm to (95.5, 61.0)
- moved R7 73.4 mm to (97.8, 60.7)
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Connections:
- net /CAN_RS renamed Net-(U5-Rs)
- net /CAN_RXD renamed Net-(JP3-A)
- net /DRV_CPH renamed Net-(U2-CPH)
- net /DRV_CPL renamed Net-(U2-CPL)
- net /DRV_VCP renamed Net-(U2-VCP)
- C2 pad 1: Net-(U4-SW) -> Net-(U4-BOOT)
- C2 pad 2: Net-(U4-BST) -> Net-(U4-SW)
- TP1 pad 1: /EXP_IO12 -> /EXP_IO5
- TP2 pad 1: /EXP_IO13 -> /EXP_IO6
- U1 pad 10: /MAG_SCL -> /DRV_nFAULT
- U1 pad 11: /MAG_INT -> /DRV_nSLEEP
- U1 pad 12: /EXP_IO12 -> /DRV_IN2_PH
- U1 pad 13: /EXP_IO13 -> /DRV_IN1_EN
- U1 pad 2: /DRV_nFAULT -> /MAG_SDA
- U1 pad 3: /SDA_CANTX -> /MAG_SCL
- U1 pad 4: /SCL_CANRX -> /MAG_INT
- U1 pad 5: /DRV_nSLEEP -> /EXP_IO5
- U1 pad 6: /DRV_IN2_PH -> /EXP_IO6
- U1 pad 7: /DRV_IN1_EN -> /EXP_IO7
- U1 pad 8: unconnected-(U1-GPIO8-Pad8) -> /SCL_CANRX
- U1 pad 9: /MAG_SDA -> /SDA_CANTX
- U1 pad RX: /EXP_RX -> unconnected-(U1-PadRX)
- U1 pad TX: /EXP_TX -> unconnected-(U1-PadTX)
- U4 pad 1: +5V -> GND
- U4 pad 2: +12V -> Net-(U4-SW)
- U4 pad 4: GND -> Net-(U4-FB)
- U4 pad 5: Net-(U4-SW) -> unconnected-(U4-EN-Pad5)
- U4 pad 6: Net-(U4-BST) -> Net-(U4-BOOT)
Routing:
- net +12V: track 52.5 -> 0.00 mm, vias 3 -> 0
- net +3V3: track 48.6 -> 0.00 mm, vias 3 -> 0
- net GND: track 38.9 -> 0.00 mm, vias 18 -> 0
- net /CANH: track 21.8 -> 0.00 mm, vias 2 -> 0
- net /BUS_N: track 17.8 -> 0.00 mm, vias 2 -> 0
- net /CANL: track 17.3 -> 0.00 mm, vias 1 -> 0
- net /DRV_IPROPI: track 16.9 -> 0.00 mm
- net /MAG_SDA: track 16.2 -> 0.00 mm
- net /EXP_IO12: track 13.4 -> 0.00 mm
- net /DRV_nFAULT: track 13.4 -> 0.00 mm
- net +5V: track 12.7 -> 0.00 mm
- net /MAG_SCL: track 12.1 -> 0.00 mm
- net /SDA_CANTX: track 11.7 -> 0.00 mm, vias 1 -> 0
- net /BUS_P: track 10.7 -> 0.00 mm, vias 2 -> 0
- net /SCL_CANRX: track 9.05 -> 0.00 mm
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Other:
- board text added: "IO5"
- board text added: "IO6"
- board text removed: "IO12"
- board text removed: "IO13"
- board text removed: "RX"
- board text removed: "TX"
