File: PCB/main-board/main-board.kicad_pcb (KiCad board)
At the start: 2 copper layers, 24.7 x 28.4 mm, 44 parts, among them CN2 XT30APB, J2 Motor (JST-PH 2P), U1 ESP32-S3-SuperMini, U2 DRV8876RGTR, U3 MLX90393SLW-ABA-011-RE, U4 TPS54202DDCR, U5 SN65HVD230

Commit message: layout
Parts:
- C14, R8, R9: moved to B.Cu
- moved C5 94.4 mm to (28.5, 23.0), turned to -90 degrees
- moved C6 90.9 mm to (25.3, 23.2)
- moved C8 90.4 mm to (31.0, 23.0), turned to -90 degrees
- moved C7 89.7 mm to (29.8, 23.0), turned to 90 degrees
- moved R2 88.1 mm to (32.5, 24.8), turned to 90 degrees
- moved D1 87.7 mm to (27.4, 35.0), turned to 180 degrees
- moved R1 82.6 mm to (25.5, 28.2)
- moved L1 82.3 mm to (31.5, 31.6), turned to 90 degrees
- moved R4 81.6 mm to (22.0, 34.5), turned to -90 degrees
- moved C12 79.4 mm to (22.8, 28.2), turned to 90 degrees
- moved C9 78.5 mm to (22.2, 41.0)
- moved U5 76.6 mm to (28.4, 33.0), turned to -90 degrees
- moved C11 76.4 mm to (23.2, 41.0)
- moved R6 74.1 mm to (29.2, 41.0)
- moved C10 74.0 mm to (24.2, 41.0), turned to -90 degrees
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Other:
- board text added: "Nothing to see here"
- board text added: "Unlocked v2 Arm PCB v1.0 By @etinaude"

Commit message: maybe placed?
Parts:
- removed JP1: D+ select, Jumper:SolderJumper-3_P1.3mm_Bridged12_RoundedPad1.0x1.5mm
- removed JP2: D- select, Jumper:SolderJumper-3_P1.3mm_Bridged12_RoundedPad1.0x1.5mm
- removed JP3: RX link, Jumper:SolderJumper-2_P1.3mm_Bridged_RoundedPad1.0x1.5mm
- JP4, TP6: moved to B.Cu
- moved TP6 17.3 mm to (32.9, 23.0)
- moved JP4 16.1 mm to (39.6, 40.4), turned to 0 degrees
- moved R5 14.3 mm to (41.8, 40.4)
- moved C13 13.0 mm to (29.3, 39.3), turned to 180 degrees
- moved D1 12.5 mm to (36.8, 26.6), turned to -90 degrees
- moved R6 6.66 mm to (27.6, 34.5), turned to 0 degrees
- moved U5 5.33 mm to (29.3, 38.2), turned to 90 degrees
- moved R2 4.81 mm to (30.0, 28.9), turned to 180 degrees
- moved C10 2.54 mm to (25.6, 38.9)
- moved R1 1.59 mm to (24.3, 29.3), turned to -90 degrees
- moved U2 0.31 mm to (30.0, 26.1)
- moved R7 0.26 mm to (32.8, 43.0)
- moved R3 0.25 mm to (26.8, 37.5)
- renumbered IO7 to TP3
Connections:
- CN2 pad 1: /BUS_N -> /CANL
- CN2 pad 2: /BUS_P -> /CANH
- R7 pad 2: /SDA_CANTX -> /CAN_TX
- U1 pad 8: /SCL_CANRX -> /CAN_TX
- U1 pad 9: /SDA_CANTX -> /CAN_RX
- U5 pad 1: /SDA_CANTX -> /CAN_TX
- U5 pad 4: Net-(JP3-A) -> /CAN_RX
Other:
- board text added: "IO7"
- board text removed: "CAN"
- board text removed: "I2C"
- board text removed: "RX CAN"

Commit message: working maybe
Parts:
- C14: value 47pF 50V -> 100pF 50V
- moved C13 0.72 mm to (28.9, 39.9)
- moved C5 0.10 mm to (28.4, 23.0)
Routing:
- net +3V3: track 0.00 -> 60.7 mm, vias 0 -> 5
- net +12V: track 0.00 -> 31.0 mm, vias 0 -> 3
- net GND: track 0.00 -> 30.6 mm, vias 0 -> 14
- net +5V: track 0.00 -> 28.7 mm
- net /CANL: track 0.00 -> 18.6 mm
- net /CANH: track 0.00 -> 17.4 mm
- net /DRV_nFAULT: track 0.00 -> 14.3 mm, vias 0 -> 1
- net /MAG_SDA: track 0.00 -> 13.7 mm
- net /CAN_TX: track 0.00 -> 11.8 mm
- net /DRV_nSLEEP: track 0.00 -> 11.2 mm, vias 0 -> 1
- net /DRV_IPROPI: track 0.00 -> 9.97 mm, vias 0 -> 2
- net /DRV_IN2_PH: track 0.00 -> 9.92 mm, vias 0 -> 1
- net /EXP_IO5: track 0.00 -> 9.45 mm
- net /DRV_IN1_EN: track 0.00 -> 8.28 mm, vias 0 -> 1
- net /MAG_SCL: track 0.00 -> 7.12 mm
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