File: PCB/main-board/main-board.kicad_sch (KiCad schematic)
At the start: 37 parts, among them J1 USB-C 16P (12V + I2C), J2 Motor (JST-PH 2P), U1 ESP32-S3-SuperMini, U2 DRV8876RGTR, U3 MLX90393SLW-ABA-011-RE, U4 AP63205WU-7

Commit message: PCB stuff
Parts:
- removed TP10, TP11: Pad, TestPoint:TestPoint_Pad_D1.0mm, symbol Connector:TestPoint
- added C13: 100nF 16V, Capacitor_SMD:C_0402_1005Metric, symbol Device:C
- added JP1: D+ select, Jumper:SolderJumper-3_P1.3mm_Bridged12_RoundedPad1.0x1.5mm, symbol Jumper:SolderJumper_3_Bridged12
- added JP2: D- select, Jumper:SolderJumper-3_P1.3mm_Bridged12_RoundedPad1.0x1.5mm, symbol Jumper:SolderJumper_3_Bridged12
- added JP3: RX link, Jumper:SolderJumper-2_P1.3mm_Bridged_RoundedPad1.0x1.5mm, symbol Jumper:SolderJumper_2_Bridged
- added JP4: 120R term, Jumper:SolderJumper-2_P1.3mm_Open_RoundedPad1.0x1.5mm, symbol Jumper:SolderJumper_2_Open
- added R5: 120R, Resistor_SMD:R_0402_1005Metric, symbol Device:R
- added R6: 10k, Resistor_SMD:R_0402_1005Metric, symbol Device:R
- added U5: SN65HVD230, Package_SO:SOIC-8_3.9x4.9mm_P1.27mm, symbol Interface_CAN_LIN:SN65HVD230
- J1: value USB-C 16P (12V + I2C) -> USB-C 16P (12V + CAN/I2C)
Connections:
- net +3V3: now also C13.1, U5.3 (VCC)
- net GND: now also C13.2, R6.2, U5.2 (GND)
- net I2C_SCL renamed BUS_N
- net BUS_N: now also JP2.2 (C); no longer U1.4 (GPIO4)
- net I2C_SDA renamed BUS_P
- net BUS_P: now also JP1.2 (C); no longer U1.3 (GPIO3)
- new net: JP4.2 (B), R5.1
- new net CANH: JP1.1 (A), JP4.1 (A), U5.7 (CANH)
- new net CANL: JP2.1 (A), R5.2, U5.6 (CANL)
- new net CAN_RS: R6.1, U5.8 (Rs)
- new net CAN_RXD: JP3.1 (A), U5.4 (R)
- new net SCL_CANRX: JP2.3 (B), JP3.2 (B), U1.4 (GPIO4)
- new net SDA_CANTX: JP1.3 (B), U1.3 (GPIO3), U5.1 (D)
- no-connect marks 7 -> 8
Other:
- note added: "12 V + CAN/I2C IN (USB-C, not USB)"
- note added: "CAN BUS (default) / I2C OPTION"
- note added: "U5 hand-soldered on top, under the SuperMini. R5, R6, C13 on the bottom (JLC). Pin map: PCB/README.md."
- note added: "USB-C reused: VBUS 12 V, D+/D- = CANH/CANL (or I2C SDA/SCL via JP1/JP2). Not USB."
- note removed: "12 V + I2C IN (USB-C, not USB)"
- note removed: "DESIGN NOTES"
- note removed: "Power, assembly and part notes: PCB/README.md."
- note removed: "USB-C reused: VBUS 12 V, D+/D- I2C. Not USB."

Commit message: PCB dev
Parts:
- removed J1: USB-C 16P (12V + CAN/I2C), main-board:USB-C_HX-TYPE-C-16PIN_NPTH-pegs, symbol main-board:HXTYPE-C16PIN
- removed TP8, TP9: Pad, TestPoint:TestPoint_Pad_D1.5mm, symbol Connector:TestPoint
- added CN2: XT30APB, main-board:CONN-TH_XT30APB, symbol main-board:XT30APB
- added R7: 10k, Resistor_SMD:R_0402_1005Metric, symbol Device:R
Connections:
- net +12V: now also CN2.4
- net +3V3: now also R7.1
- net BUS_N: now also CN2.1
- net BUS_P: now also CN2.2
- net GND: now also CN2.3
- net SDA_CANTX: now also R7.2
- no-connect marks 8 -> 4
Other:
- note added: "12 V + CAN/I2C IN - XT30 (2+2)"
- note removed: "12 V + CAN/I2C IN (USB-C, not USB)"
- note removed: "PROBE PADS"
- note removed: "USB-C reused: VBUS 12 V, D+/D- = CANH/CANL (or I2C SDA/SCL via JP1/JP2). Not USB."

Commit message: new schematic
Parts:
- removed TP4: Pad, TestPoint:TestPoint_Pad_D1.5mm, symbol Connector:TestPoint
- added C14: 47pF 50V, Capacitor_SMD:C_0402_1005Metric, symbol Device:C
- added R8: 75k, Resistor_SMD:R_0402_1005Metric, symbol Device:R
- added R9: 10k, Resistor_SMD:R_0402_1005Metric, symbol Device:R
- L1: value 4.7uH -> 10uH; LCSC Part C5832374 -> C5832376; MPN FTC252012S4R7MBCA -> FTC252012S100MBCA
- R1: value 1.5k 1% -> 3.3k; footprint Resistor_SMD:R_0402_1005Metric -> Resistor_SMD:R_0805_2012Metric_Pad1.20x1.40mm_HandSolder; LCSC Part C25867 -> C26010; MPN 0402WGF1501TCE -> 0805W8F3301T5E
- U4: value AP63205WU-7 -> TPS54202DDCR; symbol Regulator_Switching:AP63205WU -> Regulator_Switching:TPS54202DDC; LCSC Part C2071056 -> C191884; MPN AP63205WU-7 -> TPS54202DDCR; Manufacturer Diodes Incorporated -> Texas Instruments
Connections:
- net +12V: no longer U4.2 (EN)
- net +5V: now also C14.2, R8.2; no longer U4.1 (FB)
- net DRV_IN1_EN: now also U1.13 (GPIO13); no longer U1.7 (GPIO7)
- net DRV_IN2_PH: now also U1.12 (GPIO12); no longer U1.6 (GPIO6)
- net DRV_nFAULT: now also U1.10 (GPIO10); no longer U1.2 (GPIO2)
- net DRV_nSLEEP: now also U1.11 (GPIO11); no longer U1.5 (GPIO5)
- net GND: now also U4.1 (GND), R9.2; no longer U4.4 (GND)
- net MAG_INT: now also U1.4 (GPIO4); no longer U1.11 (GPIO11)
- net MAG_SCL: now also U1.3 (GPIO3); no longer U1.10 (GPIO10)
- net MAG_SDA: now also U1.2 (GPIO2); no longer U1.9 (GPIO9)
- net SCL_CANRX: now also U1.8 (GPIO8); no longer U1.4 (GPIO4)
- net SDA_CANTX: now also U1.9 (GPIO9); no longer U1.3 (GPIO3)
- net at U4.6 (BOOT): now also C2.1; no longer C2.2
- net CAN_RS: no longer names the net of R6.1, U5.8 (Rs)
- net CAN_RXD: no longer names the net of JP3.1 (A), U5.4 (R)
- net DRV_CPH: no longer names the net of C8.1, U2.11 (CPH)
- net DRV_CPL: no longer names the net of C8.2, U2.12 (CPL)
- net DRV_VCP: no longer names the net of C7.1, U2.10 (VCP)
- net EXP_IO12 renamed EXP_IO5
- net EXP_IO5: now also U1.5 (GPIO5); no longer U1.12 (GPIO12)
- net EXP_IO13 renamed EXP_IO6
- net EXP_IO6: now also U1.6 (GPIO6); no longer U1.13 (GPIO13)
- net EXP_RX: no longer names the net of U1.RX
- net EXP_TX: no longer names the net of U1.TX
- net EXP_TX: no longer TP3.1
- new net: C14.1, R8.1, R9.1, U4.4 (FB)
- new net: C2.2, L1.1, U4.2 (SW)
- new net EXP_IO7: TP3.1, U1.7 (GPIO7)
- now unconnected: U4.5 (SW)
- no-connect marks 4 -> 6
Other:
- note added: "TPS54202: VOUT = 0.596 V x (1 + R8/R9) = 5.07 V; C14 = feed-forward. EN floats (internal pull-up; 7 V max, never tie to 12 V). D1 stops USB back-feed."
- note added: "U5 hand-soldered on top, under the SuperMini. R5, R6, R7, C13 on the bottom (JLC). Pin map: PCB/README.md."
- note removed: "AP63205 fixed 5 V; D1 stops USB back-feed."
- note removed: "Centre U3 on the magnet; keep U2, U4, L1 away."
- note removed: "LAYOUT NOTES"
- note removed: "U5 hand-soldered on top, under the SuperMini. R5, R6, C13 on the bottom (JLC). Pin map: PCB/README.md."
- note removed: "Wire pads, top side. GPIOs are 3.3 V only."
- moved on the sheet: C1, C10, C11, C12, C13, C2, C3, C4, C5, C6, C7, C8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

Commit message: maybe placed?
Parts:
- removed JP1: D+ select, Jumper:SolderJumper-3_P1.3mm_Bridged12_RoundedPad1.0x1.5mm, symbol Jumper:SolderJumper_3_Bridged12
- removed JP2: D- select, Jumper:SolderJumper-3_P1.3mm_Bridged12_RoundedPad1.0x1.5mm, symbol Jumper:SolderJumper_3_Bridged12
- removed JP3: RX link, Jumper:SolderJumper-2_P1.3mm_Bridged_RoundedPad1.0x1.5mm, symbol Jumper:SolderJumper_2_Bridged
Connections:
- net BUS_N is gone; now on net CANL: CN2.1
- net BUS_P is gone; now on net CANH: CN2.2
- net CAN_RX: now reaches U5.4 (R)
- net CAN_RX: now also U1.9 (GPIO9)
- net SCL_CANRX renamed CAN_TX
- net CAN_TX: now also R7.2, U5.1 (D)
- removed net SDA_CANTX: R7.2, U1.9 (GPIO9), U5.1 (D)
Other:
- note added: "12 V + CAN IN - XT30 (2+2)"
- note added: "CAN BUS"
- note removed: "12 V + CAN/I2C IN - XT30 (2+2)"
- note removed: "CAN BUS (default) / I2C OPTION"

Commit message: working maybe
Parts:
- C14: value 47pF 50V -> 100pF 50V; LCSC Part C1567 -> C1546; MPN 0402CG470J500NT -> 0402CG101J500NT
Changed lines of the file:
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@@
 	(wire
 		(pts
-			(xy 213.36 45.72) (xy 213.36 55.88)
-		)
-		(stroke
-			(width 0)
-			(type default)
-		)
-	)
-	(wire
-		(pts
 			(xy 215.9 115.57) (xy 210.82 115.57)
 		)
@@
 	(wire
 		(pts
-			(xy 213.36 55.88) (xy 213.36 58.42)
+			(xy 213.36 45.72) (xy 213.36 58.42)
 		)
 		(stroke
@@
 			)
 		)
-		(property "Value" "47pF 50V"
+		(property "Value" "100pF 50V"
 			(at 143.51 69.85 90)
 			(show_name no)
@@
 			)
 		)
-		(property "Datasheet" "https://www.lcsc.com/product-detail/C1567.html"
+		(property "Datasheet" "https://www.lcsc.com/product-detail/C1546.html"
 			(at 143.51 66.04 90)
 			(hide yes)
@@
 			)
 		)
-		(property "Description" "Buck feed-forward across R8 (TI Table 7-2 / Eq. 16). 47pF 50V C0G 5% 0402"
+		(property "Description" "Buck feed-forward across R8 (TI Table 7-2 / Eq. 16). 100pF 50V C0G 5% 0402"
 			(at 143.51 66.04 90)
 			(hide yes)
@@
 			)
 		)
-		(property "MPN" "0402CG470J500NT"
+		(property "MPN" "0402CG101J500NT"
 			(at 143.51 66.04 90)
 			(hide yes)
@@
 			)
 		)
-		(property "LCSC Part" "C1567"
+		(property "LCSC Part" "C1546"
 			(at 143.51 66.04 90)
 			(hide yes)
